Commit message: update

File: src/turn_on_wheeltec_robot/urdf/mini_mec_robot.urdf (robot description, URDF)
Before this commit: robot wheeltec_robot, 5 links, 4 joints
Links:
- link base_link: geometry visual box size=0.296 0.296 0.003
- link left_front_link: geometry visual cylinder length=0.0372 radius=0.04
- link left_wheel_link: geometry visual cylinder length=0.0372 radius=0.04
- link right_front_link: geometry visual cylinder length=0.0372 radius=0.04
- link right_wheel_link: geometry visual cylinder length=0.0372 radius=0.04
Joints:
- joint left_front_joint: origin xyz=0.0825 0.1049 0.0375 rpy=1.57 0 0 -> xyz=0.107715 0.1344 0.04 rpy=1.57 0 0
- joint left_wheel_joint: origin xyz=-0.0825 0.1049 0.0375 rpy=1.57 0 0 -> xyz=-0.107715 0.1344 0.04 rpy=1.57 0 0
- joint right_front_joint: origin xyz=0.0825 -0.1049 0.0375 rpy=1.57 0 0 -> xyz=0.107715 -0.1344 0.04 rpy=1.57 0 0
- joint right_wheel_joint: origin xyz=-0.0825 -0.1049 0.0375 rpy=1.57 0 0 -> xyz=-0.107715 -0.1344 0.04 rpy=1.57 0 0

Commit message: motion server update

File: src/turn_on_wheeltec_robot/urdf/mini_mec_robot.urdf (robot description, URDF)
Before this commit: robot wheeltec_robot, 5 links, 4 joints
Links:
- link left_front_link: geometry visual cylinder length=0.0374 radius=0.04
- link left_wheel_link: geometry visual cylinder length=0.0374 radius=0.04
- link right_front_link: geometry visual cylinder length=0.0374 radius=0.04
- link right_wheel_link: geometry visual cylinder length=0.0374 radius=0.04
Joints:
- joint left_front_joint: origin xyz=0.107715 0.1344 0.04 rpy=1.57 0 0 -> xyz=0.107715 0.1305 0.04 rpy=1.57 0 0
- joint left_wheel_joint: origin xyz=-0.107715 0.1344 0.04 rpy=1.57 0 0 -> xyz=-0.107715 0.1305 0.04 rpy=1.57 0 0
- joint right_front_joint: origin xyz=0.107715 -0.1344 0.04 rpy=1.57 0 0 -> xyz=0.107715 -0.1305 0.04 rpy=1.57 0 0
- joint right_wheel_joint: origin xyz=-0.107715 -0.1344 0.04 rpy=1.57 0 0 -> xyz=-0.107715 -0.1305 0.04 rpy=1.57 0 0

Commit message: length

File: src/turn_on_wheeltec_robot/urdf/mini_mec_robot.urdf (robot description, URDF)
Before this commit: robot wheeltec_robot, 5 links, 4 joints
Joints:
- joint left_front_joint: origin xyz=0.107715 0.1305 0.04 rpy=1.57 0 0 -> xyz=0.107715 0.13355 0.04 rpy=1.57 0 0
- joint left_wheel_joint: origin xyz=-0.107715 0.1305 0.04 rpy=1.57 0 0 -> xyz=-0.107715 0.13355 0.04 rpy=1.57 0 0
- joint right_front_joint: origin xyz=0.107715 -0.1305 0.04 rpy=1.57 0 0 -> xyz=0.107715 -0.13355 0.04 rpy=1.57 0 0
- joint right_wheel_joint: origin xyz=-0.107715 -0.1305 0.04 rpy=1.57 0 0 -> xyz=-0.107715 -0.13355 0.04 rpy=1.57 0 0

Commit message: new car

File: src/turn_on_wheeltec_robot/urdf/mini_mec_robot.urdf (robot description, URDF)
Before this commit: robot wheeltec_robot, 5 links, 4 joints
Links:
- link base_link: geometry visual box size=0.28 0.26 0.006
- link left_front_link: geometry visual cylinder length=0.042 radius=0.0385
- link left_wheel_link: geometry visual cylinder length=0.042 radius=0.0385
- link right_front_link: geometry visual cylinder length=0.042 radius=0.0385
- link right_wheel_link: geometry visual cylinder length=0.042 radius=0.0385
Joints:
- joint left_front_joint: origin xyz=0.107715 0.13355 0.04 rpy=1.57 0 0 -> xyz=0.096 0.1145 0.0385 rpy=1.57 0 0
- joint left_wheel_joint: origin xyz=-0.107715 0.13355 0.04 rpy=1.57 0 0 -> xyz=-0.096 0.1145 0.0385 rpy=1.57 0 0
- joint right_front_joint: origin xyz=0.107715 -0.13355 0.04 rpy=1.57 0 0 -> xyz=0.096 -0.1145 0.0385 rpy=1.57 0 0
- joint right_wheel_joint: origin xyz=-0.107715 -0.13355 0.04 rpy=1.57 0 0 -> xyz=-0.096 -0.1145 0.0385 rpy=1.57 0 0

Commit message: pal

File: src/turn_on_wheeltec_robot/urdf/mini_mec_robot.urdf (robot description, URDF)
Before this commit: robot wheeltec_robot, 5 links, 4 joints
Joints:
- joint left_front_joint: origin xyz=0.096 0.1145 0.0385 rpy=1.57 0 0 -> xyz=0.096 0.1045 0.0385 rpy=1.57 0 0
- joint left_wheel_joint: origin xyz=-0.096 0.1145 0.0385 rpy=1.57 0 0 -> xyz=-0.096 0.1045 0.0385 rpy=1.57 0 0
- joint right_front_joint: origin xyz=0.096 -0.1145 0.0385 rpy=1.57 0 0 -> xyz=0.096 -0.1045 0.0385 rpy=1.57 0 0
- joint right_wheel_joint: origin xyz=-0.096 -0.1145 0.0385 rpy=1.57 0 0 -> xyz=-0.096 -0.1045 0.0385 rpy=1.57 0 0
